Commit message: Added lidar box and lidar.

File: urdf/bringup.urdf.xacro (robot description, xacro)
@@ -3,6 +3,7 @@
     <xacro:include filename="properties.xacro"/>
     <xacro:include filename="inertia_macros.xacro"/>
-    <xacro:include filename="base.xacro"/>
+    <xacro:include filename="chassis_box.xacro"/>
     <xacro:include filename="wheels.xacro"/>
+    <xacro:include filename="lidar_box.xacro"/>
     <xacro:include filename="gazebo_plugins.xacro"/>
 </robot>

File: urdf/gazebo_plugins.xacro (robot description, xacro)
@@ -20,3 +20,28 @@
         </plugin>
     </gazebo>
+    <gazebo reference="lidar_link">
+        <sensor name="lidar_link" type="gpu_lidar">
+            <pose>0 0 0 0 0 0</pose>
+            <always_on>true</always_on>
+            <visualize>true</visualize>
+            <update_rate>30</update_rate>
+            <topic>scan</topic>
+            <!-- <gz_frame_id>lidar_link</gz_frame_id> -->
+            <lidar>
+                <scan>
+                    <horizontal>
+                        <samples>360</samples>
+                        <resolution>1</resolution>
+                        <max_angle>3.14159</max_angle>
+                        <min_angle>-3.14159</min_angle>
+                    </horizontal>
+                </scan>
+                <range>
+                    <max>10.0</max>
+                    <min>0.12</min>
+                    <resolution>0.01</resolution>
+                </range>
+            </lidar>
+        </sensor>
+    </gazebo>
 </robot>

File: urdf/properties.xacro (robot description, xacro)
@@ -12,3 +12,10 @@
     <xacro:property name="caster_mass" value="0.1"/>
     <xacro:property name="caster_radius" value="0.07"/>
+    <xacro:property name="lidar_box_mass" value="1.0"/>
+    <xacro:property name="lidar_box_length" value="0.25"/>
+    <xacro:property name="lidar_box_width" value="0.25"/>
+    <xacro:property name="lidar_box_height" value="0.1"/>
+    <xacro:property name="lidar_mass" value="1.0"/>
+    <xacro:property name="lidar_height" value="0.01"/>
+    <xacro:property name="lidar_radius" value="0.07"/>
 </robot>
