Commit message: Added separation for support wheels.

File: urdf/gazebo_plugins.xacro (robot description, xacro)
@@ -45,3 +45,11 @@
         </sensor>
     </gazebo>
+    <gazebo reference="front_caster_link">
+        <mu1>0.00000001</mu1>
+        <mu2>0.00000001</mu2>
+    </gazebo>
+    <gazebo reference="rear_caster_link">
+        <mu1>0.00000001</mu1>
+        <mu2>0.00000001</mu2>
+    </gazebo>
 </robot>

File: urdf/properties.xacro (robot description, xacro)
@@ -9,7 +9,8 @@
     <xacro:property name="wheel_height" value="0.05"/>
     <xacro:property name="wheel_radius" value="0.07"/>
-    <xacro:property name="wheel_separation" value="0.25"/>
-    <xacro:property name="caster_mass" value="0.1"/>
-    <xacro:property name="caster_radius" value="0.07"/>
+    <xacro:property name="wheel_separation" value="0.4"/>
+    <xacro:property name="support_wheel_mass" value="0.1"/>
+    <xacro:property name="support_wheel_radius" value="0.069"/>
+    <xacro:property name="support_wheel_separation" value="0.2"/>
     <xacro:property name="lidar_box_mass" value="1.0"/>
     <xacro:property name="lidar_box_length" value="0.25"/>

File: urdf/wheels.xacro (robot description, xacro)
@@ -12,5 +12,6 @@
             <collision>
                 <geometry>
-                    <cylinder radius="${wheel_radius}" length="${wheel_height}"/>
+                    <!-- <cylinder radius="${wheel_radius}" length="${wheel_height}"/> -->
+                    <sphere radius="${wheel_radius}"/>
                 </geometry>
                 <origin xyz="0 0 0" rpy="${pi / 2.0} 0 0"/>
@@ -19,9 +20,9 @@
         </link>
     </xacro:macro>
-    <xacro:macro name="caster_link" params="prefix">
-        <link name="${prefix}_caster_link">
+    <xacro:macro name="support_wheel_link" params="prefix">
+        <link name="${prefix}_support_wheel_link">
             <visual>
                 <geometry>
-                    <sphere radius="${caster_radius}"/>
+                    <sphere radius="${support_wheel_radius}"/>
                 </geometry>
                 <origin xyz="0 0 0" rpy="0 0 0"/>
@@ -29,9 +30,9 @@
             <collision>
                 <geometry>
-                    <sphere radius="${caster_radius}"/>
+                    <sphere radius="${support_wheel_radius}"/>
                 </geometry>
                 <origin xyz="0 0 0" rpy="0 0 0"/>
             </collision>
-            <xacro:inertia_of_sphere mass="${caster_mass}" radius="${caster_radius}"/>
+            <xacro:inertia_of_sphere mass="${support_wheel_mass}" radius="${support_wheel_radius}"/>
         </link>
     </xacro:macro>
@@ -44,6 +45,6 @@
         </joint>
     </xacro:macro>
-    <xacro:macro name="base_caster_joint" params="position child_name offset" >
-        <joint name="$base_${position}_caster_joint" type="fixed">
+    <xacro:macro name="base_support_wheel_joint" params="position child_name offset" >
+        <joint name="$base_${position}_support_wheel_joint" type="fixed">
             <parent link="base_link"/>
             <child link="${child_name}"/>
@@ -54,9 +55,9 @@
     <xacro:wheel_link prefix="left"/>
     <xacro:wheel_link prefix="right"/>
-    <xacro:caster_link prefix="front"/>
-    <xacro:caster_link prefix="rear"/>
+    <xacro:support_wheel_link prefix="front"/>
+    <xacro:support_wheel_link prefix="rear"/>
     <xacro:base_wheel_joint position="left" child_name="left_wheel_link" offset="${wheel_separation / 2}"/>
     <xacro:base_wheel_joint position="right" child_name="right_wheel_link" offset="${-wheel_separation / 2}"/>
-    <xacro:base_caster_joint position="front" child_name="front_caster_link" offset="${base_length / 2}"/>
-    <xacro:base_caster_joint position="rear" child_name="rear_caster_link" offset="${-base_length / 2}"/>
+    <xacro:base_support_wheel_joint position="front" child_name="front_support_wheel_link" offset="${support_wheel_separation / 2}"/>
+    <xacro:base_support_wheel_joint position="rear" child_name="rear_support_wheel_link" offset="${-support_wheel_separation / 2}"/>
 </robot>
