Commit message: Added launch arguments

File: urdf/properties.xacro (robot description, xacro)
@@ -2,13 +2,13 @@
 <robot xmlns:xacro="http://www.ros.org/wiki/xacro">
     <!-- Параметры -->
-    <xacro:property name="base_mass" value="1"/>
-    <xacro:property name="base_length" value="0.1"/>
-    <xacro:property name="base_width" value="0.1"/>
+    <xacro:property name="base_mass" value="1.0"/>
+    <xacro:property name="base_length" value="0.25"/>
+    <xacro:property name="base_width" value="0.25"/>
     <xacro:property name="base_height" value="0.1"/>
     <xacro:property name="wheel_mass" value="0.1"/>
-    <xacro:property name="wheel_height" value="0.1"/>
-    <xacro:property name="wheel_radius" value="0.1"/>
-    <xacro:property name="wheel_separation" value="0.1"/>
+    <xacro:property name="wheel_height" value="0.05"/>
+    <xacro:property name="wheel_radius" value="0.07"/>
+    <xacro:property name="wheel_separation" value="0.25"/>
     <xacro:property name="caster_mass" value="0.1"/>
-    <xacro:property name="caster_radius" value="0.01"/>
+    <xacro:property name="caster_radius" value="0.07"/>
 </robot>

Commit message: Updated README

File: urdf/properties.xacro (robot description, xacro)
@@ -1,16 +1,18 @@
 <?xml version="1.0"?>
 <robot xmlns:xacro="http://www.ros.org/wiki/xacro">
-    <!-- Параметры -->
-    <xacro:property name="base_mass" value="1.0"/>
-    <xacro:property name="base_length" value="0.25"/>
-    <xacro:property name="base_width" value="0.25"/>
-    <xacro:property name="base_height" value="0.1"/>
-    <xacro:property name="wheel_mass" value="0.1"/>
-    <xacro:property name="wheel_height" value="0.05"/>
-    <xacro:property name="wheel_radius" value="0.07"/>
-    <xacro:property name="wheel_separation" value="0.4"/>
+    <!-- Box propreties -->
+    <!-- Chassis_box -->
+    <xacro:property name="chassis_box_mass" value="1.0"/>
+    <xacro:property name="chassis_box_length" value="0.25"/>
+    <xacro:property name="chassis_box_width" value="0.25"/>
+    <xacro:property name="chassis_box_height" value="0.1"/>
+    <xacro:property name="drive_wheel_mass" value="0.1"/>
+    <xacro:property name="drive_wheel_height" value="0.05"/>
+    <xacro:property name="drive_wheel_radius" value="0.07"/>
+    <xacro:property name="drive_wheel_separation" value="0.4"/>
     <xacro:property name="support_wheel_mass" value="0.1"/>
     <xacro:property name="support_wheel_radius" value="0.069"/>
     <xacro:property name="support_wheel_separation" value="0.2"/>
+    <!-- Lidar box -->
     <xacro:property name="lidar_box_mass" value="1.0"/>
     <xacro:property name="lidar_box_length" value="0.25"/>
