Commit message: Fix alfter change name

File: urdf/chassis_box.xacro (robot description, xacro)
@@ -3,24 +3,24 @@
     <!-- Ссылки -->
     <link name="base_footprint"/>
-    <link name="base_link">
+    <link name="chassis_box_link">
         <visual>
             <geometry>
-                <box size="${base_length} ${base_width} ${base_height}"/>
+                <box size="${chassis_box_length} ${chassis_box_width} ${chassis_box_height}"/>
             </geometry>
-            <origin xyz="0 0 ${base_height / 2.0}" rpy="0 0 0"/>
+            <origin xyz="0 0 ${chassis_box_height / 2.0}" rpy="0 0 0"/>
         </visual>
         <collision>
              <geometry>
-                <box size="${base_length} ${base_width} ${base_height}"/>
+                <box size="${chassis_box_length} ${chassis_box_width} ${chassis_box_height}"/>
             </geometry>
-            <origin xyz="0 0 ${base_height / 2.0}" rpy="0 0 0"/>
+            <origin xyz="0 0 ${chassis_box_height / 2.0}" rpy="0 0 0"/>
         </collision>
-        <xacro:inertia_of_box mass="${base_mass}" length="${base_length}" width="${base_width}" height="${base_height}"/>
+        <xacro:inertia_of_box mass="${chassis_box_mass}" length="${chassis_box_length}" width="${chassis_box_width}" height="${chassis_box_height}"/>
     </link>
     <!-- Соединения -->
     <joint name="base_joint" type="fixed">
         <parent link="base_footprint"/>
-        <child link="base_link"/>
-        <origin xyz="0 0 ${wheel_radius}"/>
+        <child link="chassis_box_link"/>
+        <origin xyz="0 0 ${drive_wheel_radius}"/>
     </joint>
 </robot>

File: urdf/gazebo_plugins.xacro (robot description, xacro)
@@ -4,8 +4,8 @@
     <gazebo>
         <plugin filename="gz-sim-diff-drive-system" name="gz::sim::systems::DiffDrive">
-            <left_joint>base_left_wheel_joint</left_joint>
-            <right_joint>base_right_wheel_joint</right_joint>
-            <wheel_separation>${wheel_separation}</wheel_separation>
-            <wheel_radius>${wheel_radius}</wheel_radius>
+            <left_joint>chassis_box_to_left_drive_wheel_joint</left_joint>
+            <right_joint>chassis_box_to_right_drive_wheel_joint</right_joint>
+            <wheel_separation>${drive_wheel_separation}</wheel_separation>
+            <wheel_radius>${drive_wheel_radius}</wheel_radius>
             <topic>cmd_vel</topic>
             <odom_topic>odom</odom_topic>
@@ -16,6 +16,6 @@
         <plugin filename="gz-sim-joint-state-publisher-system" name="gz::sim::systems::JointStatePublisher">
             <topic>joint_states</topic>
-            <joint_name>base_left_wheel_joint</joint_name>
-            <joint_name>base_right_wheel_joint</joint_name>
+            <joint_name>chassis_box_to_left_drive_wheel_joint</joint_name>
+            <joint_name>chassis_box_to_right_drive_wheel_joint</joint_name>
         </plugin>
     </gazebo>
@@ -45,9 +45,9 @@
         </sensor>
     </gazebo>
-    <gazebo reference="front_caster_link">
+    <gazebo reference="front_support_wheel_link">
         <mu1>0.00000001</mu1>
         <mu2>0.00000001</mu2>
     </gazebo>
-    <gazebo reference="rear_caster_link">
+    <gazebo reference="rear_support_wheel_link">
         <mu1>0.00000001</mu1>
         <mu2>0.00000001</mu2>

File: urdf/lidar_box.xacro (robot description, xacro)
@@ -32,7 +32,7 @@
     </link>
     <joint name="lidar_box_base_joint" type="fixed">
-        <parent link="base_link"/>
+        <parent link="chassis_box_link"/>
         <child link="lidar_box_link"/>
-        <origin xyz="0 0 ${base_height}"/>
+        <origin xyz="0 0 ${chassis_box_height}"/>
     </joint>
     <joint name="lidar_lidar_box_joint" type="fixed">

File: urdf/wheels.xacro (robot description, xacro)
@@ -2,9 +2,9 @@
 <robot xmlns:xacro="http://www.ros.org/wiki/xacro">
     <!-- Объявление макросов -->
-    <xacro:macro name="wheel_link" params="prefix">
-        <link name="${prefix}_wheel_link">
+    <xacro:macro name="drive_wheel_link" params="prefix">
+        <link name="${prefix}_drive_wheel_link">
             <visual>
                 <geometry>
-                    <cylinder radius="${wheel_radius}" length="${wheel_height}"/>
+                    <cylinder radius="${drive_wheel_radius}" length="${drive_wheel_height}"/>
                 </geometry>
                 <origin xyz="0 0 0" rpy="${pi / 2.0} 0 0"/>
@@ -13,9 +13,9 @@
                 <geometry>
                     <!-- <cylinder radius="${wheel_radius}" length="${wheel_height}"/> -->
-                    <sphere radius="${wheel_radius}"/>
+                    <sphere radius="${drive_wheel_radius}"/>
                 </geometry>
                 <origin xyz="0 0 0" rpy="${pi / 2.0} 0 0"/>
             </collision>
-            <xacro:inertia_of_cylinder mass="${wheel_mass}" height="${wheel_height}" radius="${wheel_radius}"/>
+            <xacro:inertia_of_cylinder mass="${drive_wheel_mass}" height="${drive_wheel_height}" radius="${drive_wheel_radius}"/>
         </link>
     </xacro:macro>
@@ -37,7 +37,7 @@
         </link>
     </xacro:macro>
-    <xacro:macro name="base_wheel_joint" params="position child_name offset" >
-        <joint name="base_${position}_wheel_joint" type="continuous">
-            <parent link="base_link"/>
+    <xacro:macro name="chassis_box_to_drive_wheel_joint" params="position child_name offset" >
+        <joint name="chassis_box_to_${position}_drive_wheel_joint" type="continuous">
+            <parent link="chassis_box_link"/>
             <child link="${child_name}"/>
             <origin xyz="0 ${offset} 0"/>
@@ -45,7 +45,7 @@
         </joint>
     </xacro:macro>
-    <xacro:macro name="base_support_wheel_joint" params="position child_name offset" >
-        <joint name="$base_${position}_support_wheel_joint" type="fixed">
-            <parent link="base_link"/>
+    <xacro:macro name="chassis_box_to_support_wheel_joint" params="position child_name offset" >
+        <joint name="$chassis_box_to_${position}_support_wheel_joint" type="fixed">
+            <parent link="chassis_box_link"/>
             <child link="${child_name}"/>
             <origin xyz="${offset} 0 0"/>
@@ -53,11 +53,11 @@
     </xacro:macro>
     <!-- Вызов макросов -->
-    <xacro:wheel_link prefix="left"/>
-    <xacro:wheel_link prefix="right"/>
+    <xacro:drive_wheel_link prefix="left"/>
+    <xacro:drive_wheel_link prefix="right"/>
     <xacro:support_wheel_link prefix="front"/>
     <xacro:support_wheel_link prefix="rear"/>
-    <xacro:base_wheel_joint position="left" child_name="left_wheel_link" offset="${wheel_separation / 2}"/>
-    <xacro:base_wheel_joint position="right" child_name="right_wheel_link" offset="${-wheel_separation / 2}"/>
-    <xacro:base_support_wheel_joint position="front" child_name="front_support_wheel_link" offset="${support_wheel_separation / 2}"/>
-    <xacro:base_support_wheel_joint position="rear" child_name="rear_support_wheel_link" offset="${-support_wheel_separation / 2}"/>
+    <xacro:chassis_box_to_drive_wheel_joint position="left" child_name="left_drive_wheel_link" offset="${drive_wheel_separation / 2}"/>
+    <xacro:chassis_box_to_drive_wheel_joint position="right" child_name="right_drive_wheel_link" offset="${-drive_wheel_separation / 2}"/>
+    <xacro:chassis_box_to_support_wheel_joint position="front" child_name="front_support_wheel_link" offset="${support_wheel_separation / 2}"/>
+    <xacro:chassis_box_to_support_wheel_joint position="rear" child_name="rear_support_wheel_link" offset="${-support_wheel_separation / 2}"/>
 </robot>

Commit message: Updated launch file

File: urdf/chassis_box.xacro (robot description, xacro)
@@ -3,5 +3,5 @@
     <!-- Ссылки -->
     <link name="base_footprint"/>
-    <link name="chassis_box_link">
+    <link name="base_link">
         <visual>
             <geometry>
@@ -21,5 +21,5 @@
     <joint name="base_joint" type="fixed">
         <parent link="base_footprint"/>
-        <child link="chassis_box_link"/>
+        <child link="base_link"/>
         <origin xyz="0 0 ${drive_wheel_radius}"/>
     </joint>

File: urdf/lidar_box.xacro (robot description, xacro)
@@ -32,5 +32,5 @@
     </link>
     <joint name="lidar_box_base_joint" type="fixed">
-        <parent link="chassis_box_link"/>
+        <parent link="base_link"/>
         <child link="lidar_box_link"/>
         <origin xyz="0 0 ${chassis_box_height}"/>

File: urdf/wheels.xacro (robot description, xacro)
@@ -39,5 +39,5 @@
     <xacro:macro name="chassis_box_to_drive_wheel_joint" params="position child_name offset" >
         <joint name="chassis_box_to_${position}_drive_wheel_joint" type="continuous">
-            <parent link="chassis_box_link"/>
+            <parent link="base_link"/>
             <child link="${child_name}"/>
             <origin xyz="0 ${offset} 0"/>
@@ -47,5 +47,5 @@
     <xacro:macro name="chassis_box_to_support_wheel_joint" params="position child_name offset" >
         <joint name="$chassis_box_to_${position}_support_wheel_joint" type="fixed">
-            <parent link="chassis_box_link"/>
+            <parent link="base_link"/>
             <child link="${child_name}"/>
             <origin xyz="${offset} 0 0"/>
